File: schema/schema.brd (EAGLE design)
At the start: 44.1 x 41.9 mm, 13 parts, among them J1 CH0, J2 CH1, J3 CH2, J4 CH3, J5 Z END STOP, J6 CLEANER SERVO

Commit message: logging
Parts:
- J1: value CH0 -> FSR C0
- J2: value CH1 -> FSR C1
- J3: value CH2 -> FSR C2
- J4: value CH3 -> FSR C3
Changed lines of the file:
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@@
 </autorouter>
 <elements>
-<element name="J1" library="SRG" package="JST_B2B-PH_HEADER" value="CH0" x="6.35" y="5.08"/>
-<element name="J2" library="SRG" package="JST_B2B-PH_HEADER" value="CH1" x="16.51" y="5.08"/>
-<element name="J3" library="SRG" package="JST_B2B-PH_HEADER" value="CH2" x="27.94" y="5.08"/>
-<element name="J4" library="SRG" package="JST_B2B-PH_HEADER" value="CH3" x="38.1" y="5.08"/>
+<element name="J1" library="SRG" package="JST_B2B-PH_HEADER" value="FSR C0" x="6.35" y="5.08"/>
+<element name="J2" library="SRG" package="JST_B2B-PH_HEADER" value="FSR C1" x="16.51" y="5.08"/>
+<element name="J3" library="SRG" package="JST_B2B-PH_HEADER" value="FSR C2" x="27.94" y="5.08"/>
+<element name="J4" library="SRG" package="JST_B2B-PH_HEADER" value="FSR C3" x="38.1" y="5.08"/>
 <element name="J5" library="SRG" package="JST_B2B-PH_HEADER" value="Z END STOP" x="16.51" y="36.83"/>
 <element name="R1" library="adafruit" library_urn="urn:adsk.eagle:library:420" package="0204/5" value="3k3" x="6.35" y="11.43"/>
