File: schema/schema.sch (EAGLE design)
At the start: 13 parts, among them J1 CH0, J2 CH1, J3 CH2, J4 CH3, J5 Z END STOP, J6 CLEANER SERVO

Commit message: logging
Parts:
- J1: value CH0 -> FSR C0
- J2: value CH1 -> FSR C1
- J3: value CH2 -> FSR C2
- J4: value CH3 -> FSR C3
Changed lines of the file:
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@@
 <parts>
 <part name="R1" library="adafruit" library_urn="urn:adsk.eagle:library:420" deviceset="R-US_" device="0204/5" value="3k3"/>
-<part name="J1" library="SRG" deviceset="JST-PH_2-PIN_HEADER" device="" value="CH0"/>
+<part name="J1" library="SRG" deviceset="JST-PH_2-PIN_HEADER" device="" value="FSR C0"/>
 <part name="SUPPLY1" library="SparkFun-PowerSymbols" deviceset="VCC" device=""/>
 <part name="R2" library="adafruit" library_urn="urn:adsk.eagle:library:420" deviceset="R-US_" device="0204/5" value="3k3"/>
-<part name="J2" library="SRG" deviceset="JST-PH_2-PIN_HEADER" device="" value="CH1"/>
+<part name="J2" library="SRG" deviceset="JST-PH_2-PIN_HEADER" device="" value="FSR C1"/>
 <part name="SUPPLY2" library="SparkFun-PowerSymbols" deviceset="VCC" device=""/>
 <part name="R3" library="adafruit" library_urn="urn:adsk.eagle:library:420" deviceset="R-US_" device="0204/5" value="3k3"/>
-<part name="J3" library="SRG" deviceset="JST-PH_2-PIN_HEADER" device="" value="CH2"/>
+<part name="J3" library="SRG" deviceset="JST-PH_2-PIN_HEADER" device="" value="FSR C2"/>
 <part name="SUPPLY3" library="SparkFun-PowerSymbols" deviceset="VCC" device=""/>
 <part name="R4" library="adafruit" library_urn="urn:adsk.eagle:library:420" deviceset="R-US_" device="0204/5" value="3k3"/>
-<part name="J4" library="SRG" deviceset="JST-PH_2-PIN_HEADER" device="" value="CH3"/>
+<part name="J4" library="SRG" deviceset="JST-PH_2-PIN_HEADER" device="" value="FSR C3"/>
 <part name="SUPPLY4" library="SparkFun-PowerSymbols" deviceset="VCC" device=""/>
 <part name="GND5" library="supply1" library_urn="urn:adsk.eagle:library:371" deviceset="GND" device=""/>
